Commit message: 20210423-2

File: demo/urdf/demo_robot.urdf (robot description, URDF)
Before this commit: robot ur5e, 3 links, 2 joints
Links:
- removed link baseplate_link
- removed link mountingplate_link
- removed link world
Joints:
- removed joint baseplate_joint
- removed joint mountingplate_joint

File: demo/urdf/demo_robot.urdf.xacro (robot description, xacro)
@@ -1,48 +1,4 @@
 <?xml version="1.0"?>
 <robot xmlns:xacro="http://ros.org/wiki/xacro"
-       name="ur5e" >
-    <material name="blue">
-        <color rgba="0 0 0.8 1" />
-    </material>
-    <material name="white">
-        <color rgba="1 1 1 1" />
-    </material>
-    <material name="red">
-        <color rgba="0.8 0 0 1" />
-    </material>
-    <material name="green">
-        <color rgba="0 0.8 0 1" />
-    </material>
-    <material name="LightGrey">
-        <color rgba="0.7 0.7 0.7 1.0" />
-    </material>
-   <link name="world" />
-  <link name="baseplate_link">
-    <visual>
-      <origin xyz="0 0 0.0" />
-      <geometry>
-        <box size="1.1 0.7 0.03" />
-      </geometry>
-      <material name="LightGrey"/>
-    </visual>
-  </link>
-  <joint name="baseplate_joint" type="fixed">
-    <origin xyz="0 0 0" />
-    <parent link="world" />
-    <child link="baseplate_link" />
-  </joint>
-  <link name="mountingplate_link">
-    <visual>
-      <origin xyz="0 0 0.0" />
-      <geometry>
-        <box size="0.3 0.3 0.012" />
-      </geometry>
-      <material name="red"/>
-    </visual>
-  </link>
-  <joint name="mountingplate_joint" type="fixed">
-    <origin xyz="0.0 -0.20 0.021" />
-    <parent link="baseplate_link" />
-    <child link="mountingplate_link" />
-  </joint>
+       name="robot_model" >
 </robot>

File: demo/urdf/demo_robot_uitgewerkt.urdf.xacro (robot description, xacro)
@@ -53,10 +53,10 @@
   </joint>
   <!-- robot to mouting_plate. -->
-  <joint name="mountingplate_link" type="fixed">
+  <joint name="mountingplate_to_robot_joint" type="fixed">
     <parent link="mountingplate_link" />
     <child link="robot1_base_link" />
     <origin xyz="0.0 0.0 0.01" rpy="0.0 0.0 0.0"/>
   </joint>
-  <joint name="beugel_to_vacuum_gripper" type ="fixed">
+  <joint name="robot1_to_vacuum_gripper_joint" type ="fixed">
     <parent link="robot1_tool0" />
     <child link="vacuum_gripper_base_link" />
